Commit message: fixed xacro

File: aloha.urdf.xacro (robot description, xacro)
@@ -38,10 +38,10 @@
   </xacro:macro>
   <!-- Left Arm Example -->
-  <xacro:vx_link name="left/base_link" mesh="vx300s_1_base.stl" mass="0.969034" ixx="0.0071633" iyy="0.00602451" izz="0.00169819"/>
-  <xacro:vx_link name="left/shoulder_link" mesh="vx300s_2_shoulder.stl" mass="0.798614" ixx="0.00120156" iyy="0.00113744" izz="0.0009388"/>
+  <xacro:vx_link name="left_base_link" mesh="vx300s_1_base.stl" mass="0.969034" ixx="0.0071633" iyy="0.00602451" izz="0.00169819"/>
+  <xacro:vx_link name="left_shoulder_link" mesh="vx300s_2_shoulder.stl" mass="0.798614" ixx="0.00120156" iyy="0.00113744" izz="0.0009388"/>
   <xacro:vx_joint
-    name="left/waist"
-    parent="left/base_link"
-    child="left/shoulder_link"
+    name="left_waist"
+    parent="left_base_link"
+    child="left_shoulder_link"
     type="revolute"
     xyz="0 0 0.079"
@@ -49,10 +49,10 @@
     effort="35" velocity="1.0" damping="5.76"/>
   <!-- Right Arm Example -->
-  <xacro:vx_link name="right/base_link" mesh="vx300s_1_base.stl" mass="0.969034" ixx="0.0071633" iyy="0.00602451" izz="0.00169819"/>
-  <xacro:vx_link name="right/shoulder_link" mesh="vx300s_2_shoulder.stl" mass="0.798614" ixx="0.00120156" iyy="0.00113744" izz="0.0009388"/>
+  <xacro:vx_link name="right_base_link" mesh="vx300s_1_base.stl" mass="0.969034" ixx="0.0071633" iyy="0.00602451" izz="0.00169819"/>
+  <xacro:vx_link name="right_shoulder_link" mesh="vx300s_2_shoulder.stl" mass="0.798614" ixx="0.00120156" iyy="0.00113744" izz="0.0009388"/>
   <xacro:vx_joint
-    name="right/waist"
-    parent="right/base_link"
-    child="right/shoulder_link"
+    name="right_waist"
+    parent="right_base_link"
+    child="right_shoulder_link"
     type="revolute"
     xyz="0 0 0.079"
@@ -60,11 +60,11 @@
     effort="35" velocity="1.0" damping="5.76"/>
   <!-- Finger Coupling -->
-  <joint name="left/finger_coupling" type="fixed">
-    <parent link="left/left_finger_link"/>
-    <child link="left/right_finger_link"/>
+  <joint name="left_finger_coupling" type="fixed">
+    <parent link="left_left_finger_link"/>
+    <child link="left_right_finger_link"/>
   </joint>
-  <joint name="right/finger_coupling" type="fixed">
-    <parent link="right/left_finger_link"/>
-    <child link="right/right_finger_link"/>
+  <joint name="right_finger_coupling" type="fixed">
+    <parent link="right_left_finger_link"/>
+    <child link="right_right_finger_link"/>
   </joint>
 </xacro:robot>
